File: sch/core/core.kicad_pcb (KiCad board)
At the start: 2 copper layers, 44.8 x 72.5 mm, 68 parts, among them J1 USB_B_Micro, J10 Conn_01x08, J2 Reset, J3 V_3.3, J4 CHRG_OUT, J5 V_USB, J6 Conn_01x18, J7 Micro_SD_Card_Det, J8 Debug, J9 Conn_02x09_Odd_Even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

Commit message: makise gui add
Parts:
- moved J10 2.25 mm to (168.0, 97.8)
- moved C4 2.02 mm to (164.0, 95.2)
Routing:
- net GND: track 495.4 -> 489.4 mm
- net /C1: track 6.03 -> 8.77 mm
- net /C2: track 5.64 -> 8.35 mm
- net /C3: track 5.43 -> 7.91 mm
- net /C6: track 4.81 -> 7.06 mm
- net /C5: track 5.01 -> 7.03 mm
- net /C4: track 5.22 -> 7.22 mm
- net +3V3: track 424.9 -> 423.1 mm
- net /CRYST_1: track 17.2 -> 16.3 mm
Other:
- net class Default: clearance 0.2 -> 0.15
- net class power: clearance 0.2 -> 0.15
- rule trace_clearance: 0.2 -> 0.15
