File: sch/core/core.kicad_pcb (KiCad board)
At the start: 2 copper layers, 45 parts, among them J1 USB_B_Micro, J2 Reset, J3 V_3.3, J4 CHRG_OUT, J5 V_USB, J6 Conn_01x09, U1 STM32F427VITx, U2 LM3671-3.3, U3 BQ24296, U4 USBLC6-4SC6

Commit message: sch core done
Parts:
- added BT1: Battery_Cell, Connector_PinSocket_2.54mm:PinSocket_1x02_P2.54mm_Vertical, F.Cu at (184.0, 109.5)
- added C28: 10u, Capacitors_SMD:C_0805, F.Cu at (175.4, 107.5)
- added C29: 10u, Capacitors_SMD:C_0805, F.Cu at (177.2, 107.5)
- added C30: 10nF, Capacitors_SMD:C_0805, F.Cu at (151.0, 97.2)
- added C31: 10nF, Capacitors_SMD:C_0805, F.Cu at (153.0, 73.2)
- added C32: 30pF, Capacitors_SMD:C_0805, F.Cu at (152.0, 84.0)
- added C33: 30pF, Capacitors_SMD:C_0805, F.Cu at (152.0, 86.5)
- added C34: 10u, Capacitors_SMD:C_0805, F.Cu at (171.5, 65.0)
- added C35: 0.1u, Capacitors_SMD:C_0402, F.Cu at (173.5, 63.5)
- added C36: 10u, Capacitors_SMD:C_0805, F.Cu at (183.8, 75.5)
- added J7: Micro_SD_Card_Det, Connectors_Hirose:microSD_Card_Receptacle_Hirose_DM3AT-SF-PEJM5, F.Cu at (183.0, 62.0)
- added J8: Debug, Connector_PinHeader_1.27mm:PinHeader_1x05_P1.27mm_Vertical, F.Cu at (187.0, 78.5)
- added J9: Conn_02x09_Odd_Even, Connector_PinSocket_2.54mm:PinSocket_2x09_P2.54mm_Vertical, F.Cu at (159.6, 50.0)
- added L2: 1uH, Inductors:Inductor_Taiyo-Yuden_NR-40xx_HandSoldering, F.Cu at (176.0, 102.2)
- added Q1: BSS138, TO_SOT_Packages_SMD:SOT-23, F.Cu at (162.5, 69.0)
- added R10: 510, Resistors_SMD:R_0603, F.Cu at (157.2, 83.5)
- added R11: 510, Resistors_SMD:R_0603, F.Cu at (157.2, 85.0)
- added R7: R_BACKLIGHT, Resistors_SMD:R_0805, F.Cu at (165.5, 70.0)
- added R8: 22k, Resistors_SMD:R_0603, F.Cu at (150.0, 72.5)
- added R9: 22k, Resistors_SMD:R_0603, F.Cu at (154.0, 98.0)
- added U5: KXO-V97, Crystals:Crystal_SMD_7050-4pin_7.0x5.0mm, F.Cu at (152.0, 78.8)
- added U6: KXO-V97, Crystals:Crystal_SMD_7050-4pin_7.0x5.0mm, F.Cu at (152.0, 92.0)
- J2: footprint Connector_PinHeader_2.54mm:PinHeader_1x02_P2.54mm_Vertical -> Connector_PinHeader_1.27mm:PinHeader_1x02_P1.27mm_Vertical
- J6: value Conn_01x09 -> Conn_01x18; footprint Connector_PinHeader_2.54mm:PinHeader_1x09_P2.54mm_Vertical -> core:ILI9341_18Pin; moved to B.Cu
- moved J5 47.0 mm to (158.5, 106.2), turned to 90 degrees
- moved J6 40.5 mm to (169.6, 70.8), turned to 180 degrees
- moved C25 40.0 mm to (183.8, 79.2), turned to 270 degrees
- moved C17 39.5 mm to (162.5, 102.2)
- moved C14 38.3 mm to (167.2, 100.8), turned to 180 degrees
- moved C18 38.1 mm to (160.1, 109.0), turned to 180 degrees
- moved C21 36.3 mm to (187.0, 110.5), turned to 270 degrees
- moved C23 33.3 mm to (180.5, 111.0), turned to 270 degrees
- moved C22 33.0 mm to (178.5, 111.0), turned to 270 degrees
- moved U4 32.7 mm to (153.8, 110.5), turned to 180 degrees
- moved C26 32.6 mm to (178.2, 97.8), turned to 180 degrees
- moved C27 32.5 mm to (168.0, 67.5), turned to 180 degrees
- moved U2 30.7 mm to (188.0, 97.2), turned to 90 degrees
- moved R6 30.3 mm to (175.0, 114.0), turned to 270 degrees
- moved C3 29.9 mm to (184.5, 98.2), turned to 90 degrees
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Connections:
- J1 pad 2: /power/USB_DM -> /USB_D-
- J1 pad 3: /power/USB_DP -> /USB_D+
- J1 pad 4: /power/USB_ID -> /USB_ID
- J6 pad 1: +3V3 -> GND
- J6 pad 2: GND -> /L_RST
- J6 pad 3: /display/CS -> /L_SCK
- J6 pad 4: /display/RST -> /L_DC
- J6 pad 5: /display/DC -> /L_CS
- J6 pad 6: /display/MOSI -> /L_MOSI
- J6 pad 7: /display/SCK -> /L_MISO
- J6 pad 8: /display/LED -> GND
- J6 pad 9: /display/MISO -> +3V3
- R1 pad 1: /power/BAT_SDA -> /BAT_SDA
- R2 pad 1: /power/BAT_SCL -> /BAT_SCL
- R3 pad 1: /power/BAT_INT -> /BAT_INT
- U1 pad 1: Net-(U1-Pad1) -> /AS_SCK
- U1 pad 15: Net-(U1-Pad15) -> /CRYST_2
- U1 pad 18: Net-(U1-Pad18) -> /A_SD
- U1 pad 2: Net-(U1-Pad2) -> /AG_0
- U1 pad 26: Net-(U1-Pad26) -> /CRYST_1
- U1 pad 3: Net-(U1-Pad3) -> /AG_1
- U1 pad 4: Net-(U1-Pad4) -> /AS_MISO
- U1 pad 44: Net-(U1-Pad44) -> /BAT_PG
- U1 pad 45: Net-(U1-Pad45) -> /BAT_CE
- U1 pad 46: Net-(U1-Pad46) -> /BAT_INT
- U1 pad 47: Net-(U1-Pad47) -> /BAT_SCL
- U1 pad 48: Net-(U1-Pad48) -> /BAT_SDA
- U1 pad 5: Net-(U1-Pad5) -> /AS_MOSI
- U1 pad 51: Net-(U1-Pad51) -> /A_WS
- U1 pad 52: Net-(U1-Pad52) -> /A_SCK
- U1 pad 63: Net-(U1-Pad63) -> /A_MCK
- U1 pad 65: Net-(U1-Pad65) -> /SD_D0
- U1 pad 66: Net-(U1-Pad66) -> /SD_D1
- U1 pad 67: Net-(U1-Pad67) -> /A_MCK
- U1 pad 68: Net-(U1-Pad68) -> /D_TX
- U1 pad 69: Net-(U1-Pad69) -> /USB_ID
- U1 pad 70: Net-(U1-Pad70) -> /USB_D-
- U1 pad 71: Net-(U1-Pad71) -> /USB_D+
- U1 pad 72: Net-(U1-Pad72) -> /D_SWDIO
- U1 pad 76: Net-(U1-Pad76) -> /D_SWDCLK
- U1 pad 78: Net-(U1-Pad78) -> /SD_D2
- U1 pad 79: Net-(U1-Pad79) -> /SD_D3
- U1 pad 80: Net-(U1-Pad80) -> /SD_CLK
- U1 pad 83: Net-(U1-Pad83) -> /SD_CMD
- U1 pad 84: Net-(U1-Pad84) -> /AG_2
- U1 pad 85: Net-(U1-Pad85) -> /AG_3
- U1 pad 86: Net-(U1-Pad86) -> /AG_4
- U1 pad 87: Net-(U1-Pad87) -> /L_MOSI
- U1 pad 89: Net-(U1-Pad89) -> /L_SCK
- U1 pad 90: Net-(U1-Pad90) -> /L_MISO
- U1 pad 92: Net-(U1-Pad92) -> /AC_SCL
- U1 pad 93: Net-(U1-Pad93) -> /AC_SDA
- U1 pad 95: Net-(U1-Pad95) -> /L_CS
- U1 pad 96: Net-(U1-Pad96) -> /L_DC
- U1 pad 97: Net-(U1-Pad97) -> /L_RST
- U1 pad 98: Net-(U1-Pad98) -> /L_LED
- U3 pad 2: /power/BAT_PSEL -> +3V3
- U3 pad 3: /power/BAT_PG -> /BAT_PG
- U3 pad 5: /power/BAT_SCL -> /BAT_SCL
- U3 pad 6: /power/BAT_SDA -> /BAT_SDA
- U3 pad 7: /power/BAT_INT -> /BAT_INT
- U3 pad 8: /power/BAT_OTG -> +3V3
- U3 pad 9: /power/BAT_CE -> /BAT_CE
- U4 pad 1: /power/USB_DP -> /USB_D-
- U4 pad 3: Net-(U4-Pad3) -> /USB_D+
- U4 pad 4: /power/USB_DM -> /USB_ID
- U4 pad 6: /power/USB_ID -> Net-(U4-Pad6)
Routing:
- net GND: track 0.00 -> 468.5 mm, vias 0 -> 58
- net +3V3: track 0.00 -> 418.3 mm, vias 0 -> 5
- net +BATT: track 0.00 -> 80.4 mm
- net /USB_ID: track 0.00 -> 66.3 mm, vias 0 -> 2
- net /USB_D+: track 0.00 -> 63.9 mm, vias 0 -> 2
- net /A_MCK: track 0.00 -> 62.3 mm, vias 0 -> 1
- net /USB_D-: track 0.00 -> 61.7 mm, vias 0 -> 2
- net /A_SCK: track 0.00 -> 60.7 mm, vias 0 -> 1
- net /A_WS: track 0.00 -> 58.9 mm, vias 0 -> 1
- net /AG_2: track 0.00 -> 58.7 mm, vias 0 -> 1
- net Net-(C21-Pad1): track 0.00 -> 51.5 mm
- net /AG_3: track 0.00 -> 46.0 mm, vias 0 -> 1
- net /A_SD: track 0.00 -> 45.7 mm, vias 0 -> 1
- net /AG_4: track 0.00 -> 44.2 mm, vias 0 -> 1
- net /AC_SCL: track 0.00 -> 43.2 mm, vias 0 -> 1
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- added copper zone on B.Cu, net GND
- added copper zone on F.Cu, net GND
Other:
- board outline added: 44.8 x 72.5 mm
- net class power added: clearance 0.2, trace_width 0.5, via_dia 0.8, via_drill 0.4
- board text added: "Alexander Lutsai"
- board text added: "osfi-p v01 jan 2018"
- board text added: "osfi-p version 01 by Alexander Lutsai"

Commit message: save
Parts:
- added J10: Conn_01x08, Connector_PinHeader_1.00mm:PinHeader_1x08_P1.00mm_Vertical, F.Cu at (170.2, 97.8)
- moved C4 0.50 mm to (166.0, 95.5)
Connections:
- U1 pad 31: Net-(U1-Pad31) -> /C1
- U1 pad 32: Net-(U1-Pad32) -> /C2
- U1 pad 33: Net-(U1-Pad33) -> /C3
- U1 pad 34: Net-(U1-Pad34) -> /C4
- U1 pad 35: Net-(U1-Pad35) -> /C5
- U1 pad 36: Net-(U1-Pad36) -> /C6
Routing:
- net GND: track 468.5 -> 495.4 mm, vias 58 -> 64
- net +3V3: track 418.3 -> 424.9 mm
- net /C1: track 0.00 -> 6.03 mm
- net /C2: track 0.00 -> 5.64 mm
- net /C3: track 0.00 -> 5.43 mm
- net /C4: track 0.00 -> 5.22 mm
- net /C5: track 0.00 -> 5.01 mm
- net /C6: track 0.00 -> 4.81 mm

Commit message: pcb upd
Parts:
- removed C19: 4.7u, Capacitors_SMD:C_0805
- removed C20: 47n, Capacitors_SMD:C_0805
- removed C21, C23: 20u, Capacitors_SMD:C_1206
- removed L2: 1uH, Inductors:Inductor_Taiyo-Yuden_NR-40xx_HandSoldering
- removed R5: R, Resistors_SMD:R_0603
- removed R6: RT2, Resistors_SMD:R_0603
- removed TS1: 103 NTC Thermistor R25=10k, Connector_PinHeader_1.27mm:PinHeader_1x02_P1.27mm_Vertical
- added D1: 2A, Diode_SMD:D_2010_5025Metric, F.Cu at (180.0, 113.3)
- added F1: MF-MSMF110, Fuse:Fuse_1812_4532Metric_Pad1.30x3.40mm_HandSolder, F.Cu at (174.4, 117.9)
- added RN1: 22k, Resistor_SMD:R_Array_Concave_4x0603, F.Cu at (167.0, 57.9)
- added U7: DW01-P, Package_TO_SOT_SMD:SOT-23-6, F.Cu at (172.4, 107.4)
- added U8: 8205, Package_SO:TSSOP-8_4.4x3mm_P0.65mm, F.Cu at (179.3, 109.0)
- C12: value 1u -> 10u; footprint Capacitors_SMD:C_0805 -> Capacitor_SMD:C_0805_2012Metric
- C14: value 8.2u -> 10u; footprint Capacitors_SMD:C_0805 -> Capacitor_SMD:C_0805_2012Metric
- C16, C18, C2, C22, C25, C26, C27, C28, C29, C3, C30, C31, C32, C33, C34, C36, C5, C7: footprint Capacitors_SMD:C_0805 -> Capacitor_SMD:C_0805_2012Metric
- C17: value 20u -> 100n; footprint Capacitors_SMD:C_1206 -> Capacitor_SMD:C_0805_2012Metric
- R1: footprint Resistors_SMD:R_0603 -> Resistor_SMD:R_0603_1608Metric_Pad1.05x0.95mm_HandSolder
- R2: value 22k -> 2k; footprint Resistors_SMD:R_0603 -> Resistor_SMD:R_0603_1608Metric_Pad1.05x0.95mm_HandSolder
- R3: value 22k -> 100; footprint Resistors_SMD:R_0603 -> Resistor_SMD:R_0603_1608Metric_Pad1.05x0.95mm_HandSolder
- R4: value RT1 -> 1k; footprint Resistors_SMD:R_0603 -> Resistor_SMD:R_0603_1608Metric_Pad1.05x0.95mm_HandSolder
- U3: value BQ24296 -> MCP73831-2-OT; footprint Housings_DFN_QFN:QFN-24_4x4mm_Pitch0.5mm -> Package_TO_SOT_SMD:SOT-23-5
- U4: footprint TO_SOT_Packages_SMD:SOT-23-6 -> Package_TO_SOT_SMD:SOT-23-6
- moved R1 54.5 mm to (170.9, 56.4), turned to 0 degrees
- moved R3 26.6 mm to (194.9, 107.3), turned to 0 degrees
- moved C17 26.0 mm to (188.2, 106.3), turned to 90 degrees
- moved C14 14.6 mm to (168.5, 115.3), turned to 0 degrees
- moved C12 14.0 mm to (153.6, 113.0), turned to 0 degrees
- moved C28 13.5 mm to (188.7, 109.8), turned to 0 degrees
- moved C29 13.1 mm to (164.3, 105.3)
- moved C22 13.1 mm to (169.3, 101.8), turned to 0 degrees
- moved R4 10.1 mm to (173.1, 103.1), turned to 180 degrees
- moved BT1 9.43 mm to (179.7, 117.9), turned to 90 degrees
- moved C18 5.06 mm to (157.0, 113.0), turned to 0 degrees
- moved U3 3.51 mm to (168.7, 111.1), turned to 270 degrees
- moved J5 3.43 mm to (160.1, 109.3)
- moved R2 3.39 mm to (167.3, 107.5), turned to 0 degrees
- moved U4 1.74 mm to (153.8, 108.8), turned to 0 degrees
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Connections:
- BT1 pad 1: +BATT -> Net-(BT1-Pad1)
- BT1 pad 2: GND -> Net-(BT1-Pad2)
- C14 pad 1: Net-(C14-Pad1) -> VBUS
- C17 pad 1: VBUS -> Net-(C17-Pad1)
- C17 pad 2: GND -> Net-(BT1-Pad2)
- C28 pad 1: Net-(C21-Pad1) -> +BATT
- C29 pad 1: Net-(C21-Pad1) -> +BATT
- J4 pad 1: Net-(C21-Pad1) -> +BATT
- R1 pad 1: /BAT_SDA -> +3V3
- R1 pad 2: +3V3 -> /SD_D1
- R2 pad 1: /BAT_SCL -> Net-(R2-Pad1)
- R2 pad 2: +3V3 -> GND
- R3 pad 1: /BAT_INT -> +BATT
- R3 pad 2: +3V3 -> Net-(C17-Pad1)
- R4 pad 1: Net-(C19-Pad1) -> GND
- U3 pad 1: VBUS -> /BAT_CE
- U3 pad 2: +3V3 -> GND
- U3 pad 3: /BAT_PG -> +BATT
- U3 pad 4: Net-(U3-Pad4) -> VBUS
- U3 pad 5: /BAT_SCL -> Net-(R2-Pad1)
Routing:
- net GND: track 495.4 -> 335.2 mm, vias 64 -> 44
- net +BATT: track 80.4 -> 9.35 mm
- net Net-(C21-Pad1): track 51.5 -> 0.00 mm
- net +3V3: track 424.9 -> 378.1 mm, vias 5 -> 4
- net /USB_ID: track 66.3 -> 26.6 mm, vias 2 -> 1
- net /USB_D+: track 63.9 -> 25.9 mm, vias 2 -> 1
- net /USB_D-: track 61.7 -> 24.3 mm, vias 2 -> 1
- net Net-(J1-Pad1): track 31.2 -> 0.00 mm, vias 2 -> 0
- net /BAT_CE: track 30.6 -> 0.00 mm, vias 2 -> 0
- net /BAT_INT: track 27.5 -> 0.00 mm, vias 2 -> 0
- net /BAT_SCL: track 24.4 -> 0.00 mm, vias 2 -> 0
- net /BAT_SDA: track 24.2 -> 0.00 mm, vias 2 -> 0
- net /BAT_PG: track 21.6 -> 0.00 mm, vias 2 -> 0
- net VBUS: track 15.7 -> 0.00 mm
- net Net-(C19-Pad1): track 13.6 -> 0.00 mm, vias 2 -> 0
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