File: sch/core/core.kicad_pcb (KiCad board)
At the start: 2 copper layers, 44.8 x 72.5 mm, 65 parts, among them J1 USB_B_Micro, J10 Conn_01x08, J2 Reset, J3 V_3.3, J4 CHRG_OUT, J5 V_USB, J6 Conn_01x18, J7 Micro_SD_Card_Det, J8 Debug, J9 Conn_02x09_Odd_Even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

Commit message: PCB v.2 completed
Parts:
- added R5: 22k, Resistors_SMD:R_0603_HandSoldering, F.Cu at (172.0, 68.7)
- J10: value Conn_01x08 -> Conn_01x12; footprint Connector_PinHeader_1.00mm:PinHeader_1x08_P1.00mm_Vertical -> core:conn_1_12
- moved C28 20.4 mm to (168.7, 113.8), turned to 180 degrees
- moved R4 15.3 mm to (184.9, 112.8), turned to 90 degrees
- moved C12 15.1 mm to (165.4, 103.6)
- moved U7 13.7 mm to (185.9, 109.2), turned to 0 degrees
- moved R1 12.6 mm to (173.4, 68.8), turned to 90 degrees
- moved C29 11.3 mm to (175.5, 106.2), turned to 180 degrees
- moved C18 11.2 mm to (165.4, 105.7)
- moved C14 8.47 mm to (162.8, 109.0), turned to 270 degrees
- moved J5 8.02 mm to (153.2, 105.3)
- moved R3 7.90 mm to (189.2, 112.8), turned to 90 degrees
- moved C22 7.17 mm to (169.9, 108.9), turned to 270 degrees
- moved RN1 6.61 mm to (167.9, 64.5), turned to 180 degrees
- moved R2 4.79 mm to (165.1, 111.8)
- moved U3 3.16 mm to (166.4, 109.0), turned to 180 degrees
- moved C17 2.62 mm to (189.2, 108.7)
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Connections:
- J10 pad 1: /C6 -> Net-(J10-Pad1)
- J10 pad 2: /C5 -> Net-(J10-Pad2)
- J10 pad 3: /C4 -> Net-(J10-Pad3)
- J10 pad 4: /C3 -> Net-(J10-Pad4)
- J10 pad 5: /C2 -> /C6
- J10 pad 6: /C1 -> /C5
- J10 pad 7: GND -> /C4
- J10 pad 8: +3V3 -> /C3
- RN1 pad 1: /SD_D2 -> Net-(RN1-Pad1)
- RN1 pad 2: /SD_D3 -> /SD_CMD
- RN1 pad 3: /SD_CMD -> /SD_D3
- RN1 pad 4: /SD_D0 -> /SD_D2
Routing:
- net +BATT: track 9.35 -> 122.5 mm, vias 0 -> 2
- net +3V3: track 365.8 -> 453.7 mm, vias 4 -> 6
- net /USB_ID: track 26.6 -> 57.7 mm, vias 1 -> 2
- net Net-(J1-Pad1): track 0.00 -> 31.0 mm
- net Net-(BT1-Pad2): track 12.6 -> 43.1 mm
- net GND: track 335.2 -> 365.0 mm, vias 44 -> 59
- net /USB_D+: track 25.9 -> 53.0 mm, vias 1 -> 2
- net /USB_D-: track 24.3 -> 49.5 mm, vias 1 -> 2
- net /BAT_CE: track 0.00 -> 22.5 mm, vias 0 -> 2
- net VBUS: track 0.00 -> 15.1 mm
- net Net-(U7-Pad3): track 0.00 -> 14.1 mm
- net /SD_D2: track 20.8 -> 29.5 mm
- net /SD_D3: track 19.5 -> 27.8 mm
- net Net-(R4-Pad2): track 0.00 -> 4.67 mm
- net Net-(C17-Pad1): track 0.00 -> 4.63 mm
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