File: sch/core/core.sch (KiCad schematic (older format))
At the start: 1 part, among them U1 STM32F427VITx

Commit message: sch wip
Parts:
- U1: footprint Package_QFP:LQFP-100_14x14mm_P0.5mm -> Housings_QFP:LQFP-100_14x14mm_Pitch0.5mm
Changed lines of the file:
@@
 $Descr A4 11693 8268
 encoding utf-8
-Sheet 1 2
+Sheet 1 3
 Title ""
 Date ""
@@
 F 0 "U1" H 4300 3965 50  0000 C CNN
 F 1 "STM32F427VITx" H 4300 3874 50  0000 C CNN
-F 2 "Package_QFP:LQFP-100_14x14mm_P0.5mm" H 5100 1900 50  0001 R CNN
+F 2 "Housings_QFP:LQFP-100_14x14mm_Pitch0.5mm" H 5100 1900 50  0001 R CNN
 F 3 "http://www.st.com/st-web-ui/static/active/en/resource/technical/document/datasheet/DM00071990.pdf" H 4350 3000 50  0001 C CNN
 	1    4300 2950
@@
 F 0 "U1" H 6650 3965 50  0000 C CNN
 F 1 "STM32F427VITx" H 6650 3874 50  0000 C CNN
-F 2 "Package_QFP:LQFP-100_14x14mm_P0.5mm" H 7450 1900 50  0001 R CNN
+F 2 "Housings_QFP:LQFP-100_14x14mm_Pitch0.5mm" H 7450 1900 50  0001 R CNN
 F 3 "http://www.st.com/st-web-ui/static/active/en/resource/technical/document/datasheet/DM00071990.pdf" H 6700 3000 50  0001 C CNN
 	2    6650 2950
@@
 F 0 "U1" H 1606 3965 50  0000 C CNN
 F 1 "STM32F427VITx" H 1606 3874 50  0000 C CNN
-F 2 "Package_QFP:LQFP-100_14x14mm_P0.5mm" H 2300 1900 50  0001 R CNN
+F 2 "Housings_QFP:LQFP-100_14x14mm_Pitch0.5mm" H 2300 1900 50  0001 R CNN
 F 3 "http://www.st.com/st-web-ui/static/active/en/resource/technical/document/datasheet/DM00071990.pdf" H 1550 3000 50  0001 C CNN
 	3    1500 2950
@@
 $EndComp
 $Sheet
-S 3450 5600 900  650
+S 3450 5600 1100 800
 U 5C3BFBF8
 F0 "power" 50
 F1 "power.sch" 50
-F2 "BAT_INT" I R 4350 5700 50
+F2 "BAT_INT" I R 4550 5700 50
+F3 "BAT_SDA" B R 4550 5800 50
+F4 "BAT_SCL" I R 4550 5900 50
+F5 "BAT_OTG" I R 4550 6000 50
+F6 "BAT_CE" I R 4550 6100 50
+F7 "BAT_PSEL" I R 4550 6200 50
+F8 "BAT_PG" I R 4550 6300 50
+F9 "USB_ID" B L 3450 5700 50
+F10 "USB_DM" B L 3450 5800 50
+F11 "USB_DP" B L 3450 5900 50
+$EndSheet
+$Sheet
+S 6050 5600 650  800
+U 5C4DC24C
+F0 "display" 50
+F1 "display.sch" 50
+F2 "MISO" I L 6050 5700 50
+F3 "LED" I L 6050 5800 50
+F4 "SCK" I L 6050 5900 50
+F5 "MOSI" I L 6050 6000 50
+F6 "DC" I L 6050 6100 50
+F7 "RST" I L 6050 6200 50
+F8 "CS" I L 6050 6300 50
 $EndSheet
 $EndSCHEMATC

Commit message: sch core done
Parts:
- added C34, C36: 10u, Capacitors_SMD:C_0805, symbol Device:C
- added C35: 0.1u, Capacitors_SMD:C_0402, symbol Device:C
- added J7: Micro_SD_Card_Det, Connectors_Hirose:microSD_Card_Receptacle_Hirose_DM3AT-SF-PEJM5, symbol Connector:Micro_SD_Card_Det
- added J8: Debug, Connector_PinHeader_1.27mm:PinHeader_1x05_P1.27mm_Vertical, symbol Connector_Generic:Conn_01x05
- added J9: Conn_02x09_Odd_Even, Connector_PinSocket_2.54mm:PinSocket_2x09_P2.54mm_Vertical, symbol Connector_Generic:Conn_02x09_Odd_Even
Connections:
- net CRYST_2: now reaches U1.15 (PC0)
- net A_SD: now reaches U1.18 (PC3)
- net A_SD: now also J9.1 (Pin_1)
- net A_MCK: now reaches U1.63 (PC6)
- net A_MCK: now also U1.67 (PA8), J9.4 (Pin_4)
- net SD_D0: now reaches U1.65 (PC8)
- net SD_D0: now also J7.7 (DAT0)
- net SD_D1: now reaches U1.66 (PC9)
- net SD_D1: now also J7.8 (DAT1)
- net SD_D2: now reaches U1.78 (PC10)
- net SD_D2: now also J7.1 (DAT2)
- net SD_D3: now reaches U1.79 (PC11)
- net SD_D3: now also J7.2 (DAT3/CD)
- net SD_CLK: now reaches U1.80 (PC12)
- net SD_CLK: now also J7.5 (CLK)
- net SD_CMD: now reaches U1.83 (PD2)
- net SD_CMD: now also J7.3 (CMD)
- net AG_2: now reaches U1.84 (PD3)
- net AG_2: now also J9.14 (Pin_14)
- net AG_3: now reaches U1.85 (PD4)
- net AG_3: now also J9.13 (Pin_13)
- net AG_4: now reaches U1.86 (PD5)
- net AG_4: now also J9.12 (Pin_12)
- net L_MOSI: now reaches U1.87 (PD6)
- net AS_SCK: now reaches U1.1 (PE2)
- net AS_SCK: now also J9.9 (Pin_9)
- net AG_0: now reaches U1.2 (PE3)
- net AG_0: now also J9.8 (Pin_8)
- net AG_1: now reaches U1.3 (PE4)
- net AG_1: now also J9.7 (Pin_7)
- net AS_MISO: now reaches U1.4 (PE5)
- net AS_MISO: now also J9.6 (Pin_6)
- net BAT_PG: now reaches U1.44 (PE13)
- net BAT_CE: now reaches U1.45 (PE14)
- net BAT_INT: now reaches U1.46 (PE15)
- net BAT_SCL: now reaches U1.47 (PB10)
- net BAT_SDA: now reaches U1.48 (PB11)
- net AS_MOSI: now reaches U1.5 (PE6)
- net AS_MOSI: now also J9.5 (Pin_5)
- net A_WS: now reaches U1.51 (PB12)
- net A_WS: now also J9.2 (Pin_2)
- net A_SCK: now reaches U1.52 (PB13)
- net A_SCK: now also J9.3 (Pin_3)
- net L_SCK: now reaches U1.89 (PB3)
- net L_MISO: now reaches U1.90 (PB4)
- net AC_SCL: now reaches U1.92 (PB6)
- net AC_SCL: now also J9.11 (Pin_11)
- net AC_SDA: now reaches U1.93 (PB7)
- net AC_SDA: now also J9.10 (Pin_10)
- net L_CS: now reaches U1.95 (PB8)
- net L_DC: now reaches U1.96 (PB9)
- net L_RST: now reaches U1.97 (PE0)
- net L_LED: now reaches U1.98 (PE1)
- net CRYST_1: now reaches U1.26 (PA3)
- net D_TX: now reaches U1.68 (PA9)
- net D_TX: now also J8.4 (Pin_4)
- net USB_ID: now reaches U1.69 (PA10)
- net USB_D-: now reaches U1.70 (PA11)
- net USB_D+: now reaches U1.71 (PA12)
- net D_SWDIO: now reaches U1.72 (PA13)
- net D_SWDIO: now also J8.3 (Pin_3)
- net D_SWDCLK: now reaches U1.76 (PA14)
- net D_SWDCLK: now also C36.1, J8.1 (Pin_1)
- new net +3V3: C34.1, C35.1, J7.4 (VDD), J9.18 (Pin_18)
- new net +BATT: J9.17 (Pin_17)
- new net GND: C34.2, C35.2, C36.2, J7.11 (SHIELD), J7.6 (VSS), J8.2 (Pin_2), J9.15 (Pin_15), J9.16 (Pin_16)
- no-connect marks 0 -> 40
Other:
- moved on the sheet: U1A, U1B

Commit message: save
Parts:
- added J10: Conn_01x08, Connector_PinHeader_1.00mm:PinHeader_1x08_P1.00mm_Vertical, symbol Connector_Generic:Conn_01x08
Connections:
- net +3V3: now also J10.8 (Pin_8)
- net GND: now also J10.7 (Pin_7)
- net C3: now reaches U1.33 (PC4)
- net C3: now also J10.4 (Pin_4)
- net C4: now reaches U1.34 (PC5)
- net C4: now also J10.3 (Pin_3)
- net C5: now reaches U1.35 (PB0)
- net C5: now also J10.2 (Pin_2)
- net C6: now reaches U1.36 (PB1)
- net C6: now also J10.1 (Pin_1)
- net C1: now reaches U1.31 (PA6)
- net C1: now also J10.6 (Pin_6)
- net C2: now reaches U1.32 (PA7)
- net C2: now also J10.5 (Pin_5)
- no-connect marks 40 -> 34
Changed lines of the file:
@@
 NoConn ~ 2400 2600
 NoConn ~ 2400 2700
-NoConn ~ 2400 2800
-NoConn ~ 2400 2900
 NoConn ~ 2400 3700
 NoConn ~ 4050 3100
@@
 NoConn ~ 5850 3600
 NoConn ~ 5850 3700
-NoConn ~ 5850 2700
-NoConn ~ 5850 2600
 Text Label 5950 2800 0    50   ~ 0
 A_MCK
@@
 NoConn ~ 7400 3300
 NoConn ~ 7400 3400
-NoConn ~ 9200 2200
-NoConn ~ 9200 2300
 NoConn ~ 9200 2400
 NoConn ~ 9200 3600
@@
 Wire Wire Line
 	2400 2500 3200 2500
-Wire Bus Line
-	6750 3950 10100 3950
-Wire Bus Line
-	6750 1750 6750 3950
-Wire Bus Line
-	10100 1750 10100 3950
-Wire Bus Line
-	8150 4050 8150 6500
-Wire Bus Line
-	3300 1750 3300 6500
 Entry Wire Line
 	3200 2500 3300 2600
 Text Label 2500 2500 0    50   ~ 0
 CRYST_1
+Wire Wire Line
+	2550 5700 3200 5700
+Wire Wire Line
+	2550 5800 3200 5800
+Wire Wire Line
+	2550 5900 3200 5900
+Wire Wire Line
+	2550 6000 3200 6000
+Wire Wire Line
+	2550 6100 3200 6100
+Wire Wire Line
+	2550 6200 3200 6200
+$Comp
+L power:GND #PWR0146
+U 1 1 5C506B0F
+P 2950 5400
+F 0 "#PWR0146" H 2950 5150 50  0001 C CNN
+F 1 "GND" H 2955 5227 50  0000 C CNN
+F 2 "" H 2950 5400 50  0001 C CNN
+F 3 "" H 2950 5400 50  0001 C CNN
+	1    2950 5400
+	1    0    0    -1
+$EndComp
+$Comp
+L Connector_Generic:Conn_01x08 J10
+U 1 1 5C510D95
+P 2350 5900
+F 0 "J10" H 2270 5275 50  0000 C CNN
+F 1 "Conn_01x08" H 2270 5366 50  0000 C CNN
+F 2 "Connector_PinHeader_1.00mm:PinHeader_1x08_P1.00mm_Vertical" H 2350 5900 50  0001 C CNN
+F 3 "~" H 2350 5900 50  0001 C CNN
+	1    2350 5900
+	-1   0    0    1
+$EndComp
+$Comp
+L power:+3.3V #PWR0147
+U 1 1 5C52548A
+P 2750 5450
+F 0 "#PWR0147" H 2750 5300 50  0001 C CNN
+F 1 "+3.3V" H 2765 5623 50  0000 C CNN
+F 2 "" H 2750 5450 50  0001 C CNN
+F 3 "" H 2750 5450 50  0001 C CNN
+	1    2750 5450
+	1    0    0    -1
+$EndComp
+Entry Wire Line
+	3200 5700 3300 5800
+Entry Wire Line
+	3200 5800 3300 5900
+Entry Wire Line
+	3200 5900 3300 6000
+Entry Wire Line
+	3200 6000 3300 6100
+Entry Wire Line
+	3200 6100 3300 6200
+Entry Wire Line
+	3200 6200 3300 6300
+Text Label 2650 5700 0    50   ~ 0
+C1
+Text Label 2650 5800 0    50   ~ 0
+C2
+Text Label 2650 5900 0    50   ~ 0
+C3
+Text Label 2650 6000 0    50   ~ 0
+C4
+Text Label 2650 6100 0    50   ~ 0
+C5
+Text Label 2650 6200 0    50   ~ 0
+C6
+Wire Wire Line
+	2400 2900 3200 2900
+Wire Wire Line
+	2400 2800 3200 2800
+Entry Wire Line
+	3200 2800 3300 2900
+Entry Wire Line
+	3200 2900 3300 3000
+Text Label 2500 2800 0    50   ~ 0
+C1
+Text Label 2500 2900 0    50   ~ 0
+C2
+Wire Wire Line
+	5850 2600 6650 2600
+Entry Wire Line
+	6650 2600 6750 2700
+Text Label 5950 2600 0    50   ~ 0
+C3
+Wire Wire Line
+	5850 2700 6650 2700
+Entry Wire Line
+	6650 2700 6750 2800
+Text Label 5950 2700 0    50   ~ 0
+C4
+Wire Wire Line
+	9200 2200 10000 2200
+Wire Wire Line
+	9200 2300 10000 2300
+Entry Wire Line
+	10000 2300 10100 2400
+Entry Wire Line
+	10000 2200 10100 2300
+Text Label 9250 2200 0    50   ~ 0
+C5
+Text Label 9250 2300 0    50   ~ 0
+C6
+Wire Wire Line
+	2750 5450 2750 5500
+Wire Wire Line
+	2750 5500 2550 5500
+Wire Wire Line
+	2950 5400 2950 5350
+Wire Wire Line
+	2950 5350 2850 5350
+Wire Wire Line
+	2850 5350 2850 5600
+Wire Wire Line
+	2850 5600 2550 5600
+Wire Bus Line
+	6750 3950 10100 3950
+Wire Bus Line
+	6750 1750 6750 3950
+Wire Bus Line
+	10100 1750 10100 3950
+Wire Bus Line
+	8150 4050 8150 6500
+Wire Bus Line
+	3300 1750 3300 6500
 $EndSCHEMATC

Commit message: makise gui add
Connections:
- no-connect marks 34 -> 36
Changed lines of the file:
@@
 Wire Wire Line
 	2850 5600 2550 5600
+NoConn ~ 8850 5150
+NoConn ~ 8850 5250
 Wire Bus Line
 	6750 3950 10100 3950
