File: sch/core/core.sch (KiCad schematic (older format))
At the start: 8 parts, among them J10 Conn_01x08, J7 Micro_SD_Card_Det, J8 Debug, J9 Conn_02x09_Odd_Even, U1 STM32F427VITx

Commit message: sch upd
Parts:
- added R?: 22k, symbol Device:R
- added RN?: 22k, symbol Device:R_Pack04
- U1: symbol core:STM32F427VITx -> core-rescue:STM32F427VITx-core
Connections:
- net +3V3: now also R?.1, RN?.5 (R4.2), RN?.6 (R3.2), RN?.7 (R2.2), RN?.8 (R1.2)
- net SD_CMD: now also RN?.3 (R3.1)
- net SD_D0: now also RN?.4 (R4.1)
- net SD_D1: now also R?.2
- net SD_D2: now also RN?.1 (R1.1)
- net SD_D3: now also RN?.2 (R2.1)
- no-connect marks 34 -> 36
Other:
- moved on the sheet: C34, C35, J7

Commit message: new charger schematic
Parts:
- R1: renamed from R?; footprint (none) -> Resistor_SMD:R_0603_1608Metric_Pad1.05x0.95mm_HandSolder
- RN1: renamed from RN?; footprint (none) -> Resistor_SMD:R_Array_Concave_4x0603
Changed lines of the file:
@@
 F0 "power" 50
 F1 "power.sch" 50
-F2 "BAT_INT" I R 6450 5900 50
-F3 "BAT_SDA" B R 6450 6000 50
-F4 "BAT_SCL" I R 6450 6100 50
-F5 "BAT_CE" I R 6450 5600 50
-F6 "BAT_PG" I R 6450 5800 50
-F7 "USB_ID" B R 6450 5200 50
-F8 "USB_D-" B R 6450 5300 50
-F9 "USB_D+" B R 6450 5400 50
-F10 "CRYST_2" I R 6450 6250 50
-F11 "CRYST_1" I R 6450 6350 50
+F2 "BAT_CE" I R 6450 5600 50
+F3 "USB_ID" B R 6450 5200 50
+F4 "USB_D-" B R 6450 5300 50
+F5 "USB_D+" B R 6450 5400 50
+F6 "CRYST_2" I R 6450 6250 50
+F7 "CRYST_1" I R 6450 6350 50
 $EndSheet
 $Sheet
@@
 SD_D1
 $Comp
-L Device:R_Pack04 RN?
+L Device:R_Pack04 RN1
 U 1 1 5C9222C0
 P 10600 5000
-F 0 "RN?" H 10200 5050 50  0000 L CNN
+F 0 "RN1" H 10200 5050 50  0000 L CNN
 F 1 "22k" H 10200 4950 50  0000 L CNN
-F 2 "" V 10875 5000 50  0001 C CNN
+F 2 "Resistor_SMD:R_Array_Concave_4x0603" V 10875 5000 50  0001 C CNN
 F 3 "~" H 10600 5000 50  0001 C CNN
 	1    10600 5000
@@
 	10700 5650 10700 5200
 $Comp
-L Device:R R?
+L Device:R R1
 U 1 1 5C98F98F
 P 10850 5000
-F 0 "R?" H 10920 5046 50  0000 L CNN
+F 0 "R1" H 10920 5046 50  0000 L CNN
 F 1 "22k" H 10920 4955 50  0000 L CNN
-F 2 "" V 10780 5000 50  0001 C CNN
+F 2 "Resistor_SMD:R_0603_1608Metric_Pad1.05x0.95mm_HandSolder" V 10780 5000 50  0001 C CNN
 F 3 "~" H 10850 5000 50  0001 C CNN
 	1    10850 5000
@@
 	10850 5750 10850 5150
 $Comp
-L power:+3.3V #PWR?
+L power:+3.3V #PWR0104
 U 1 1 5C99BE96
 P 10600 4650
-F 0 "#PWR?" H 10600 4500 50  0001 C CNN
+F 0 "#PWR0104" H 10600 4500 50  0001 C CNN
 F 1 "+3.3V" H 10615 4823 50  0000 C CNN
 F 2 "" H 10600 4650 50  0001 C CNN

Commit message: pcb upd
Parts:
- C34, C36: footprint Capacitors_SMD:C_0805 -> Capacitor_SMD:C_0805_2012Metric
Changed lines of the file:
@@
 F 0 "C34" H 7615 5846 50  0000 L CNN
 F 1 "10u" H 7615 5755 50  0000 L CNN
-F 2 "Capacitors_SMD:C_0805" H 7538 5650 50  0001 C CNN
+F 2 "Capacitor_SMD:C_0805_2012Metric" H 7538 5650 50  0001 C CNN
 F 3 "~" H 7500 5800 50  0001 C CNN
 	1    7500 5800
@@
 F 0 "C36" H 10815 2896 50  0000 L CNN
 F 1 "10u" H 10815 2805 50  0000 L CNN
-F 2 "Capacitors_SMD:C_0805" H 10738 2700 50  0001 C CNN
+F 2 "Capacitor_SMD:C_0805_2012Metric" H 10738 2700 50  0001 C CNN
 F 3 "~" H 10700 2850 50  0001 C CNN
 	1    10700 2850
