File: sch/core/power.sch (KiCad schematic (older format))
At the start: 57 parts, among them J1 USB_B_Micro, J2 Reset, J3 V_3.3, J4 CHRG_OUT, J5 V_USB, U1 STM32F427VITx, U2 LM3671-3.3, U3 BQ24296, U4 USBLC6-4SC6, U5 KXO-V97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

Commit message: makise gui add
Connections:
- no-connect marks 3 -> 4
Changed lines of the file:
@@
 Wire Wire Line
 	7450 5000 7950 5000
-Wire Wire Line
-	7950 5000 7950 5200
 $Comp
 L power:+3.3V #PWR0137
 U 1 1 5C680991
-P 8100 5200
-F 0 "#PWR0137" H 8100 5050 50  0001 C CNN
-F 1 "+3.3V" H 8115 5373 50  0000 C CNN
-F 2 "" H 8100 5200 50  0001 C CNN
-F 3 "" H 8100 5200 50  0001 C CNN
-	1    8100 5200
+P 8100 5150
+F 0 "#PWR0137" H 8100 5000 50  0001 C CNN
+F 1 "+3.3V" H 8115 5323 50  0000 C CNN
+F 2 "" H 8100 5150 50  0001 C CNN
+F 3 "" H 8100 5150 50  0001 C CNN
+	1    8100 5150
 	1    0    0    -1
 $EndComp
-Wire Wire Line
-	8100 5200 7950 5200
-Connection ~ 7950 5200
-Wire Wire Line
-	7950 5200 7950 5250
 $Comp
 L power:GND #PWR0138
@@
 	6250 3800 6000 3800
 Connection ~ 6000 3800
+Wire Wire Line
+	7950 5000 7950 5200
+Wire Wire Line
+	7950 5200 8100 5200
+Connection ~ 7950 5200
+Wire Wire Line
+	7950 5200 7950 5250
+Wire Wire Line
+	8100 5150 8100 5200
+$Comp
+L power:PWR_FLAG #FLG0105
+U 1 1 5C5AE97A
+P 8350 5150
+F 0 "#FLG0105" H 8350 5225 50  0001 C CNN
+F 1 "PWR_FLAG" H 8450 5300 50  0000 C CNN
+F 2 "" H 8350 5150 50  0001 C CNN
+F 3 "~" H 8350 5150 50  0001 C CNN
+	1    8350 5150
+	1    0    0    -1
+$EndComp
+Wire Wire Line
+	8350 5150 8350 5200
+Wire Wire Line
+	8350 5200 8100 5200
+Connection ~ 8100 5200
+NoConn ~ 4500 4650
 $EndSCHEMATC
