File: sch/core/power.sch (KiCad schematic (older format))
At the start: 42 parts, among them J1 USB_B_Micro, J2 Reset, U1 STM32F427VITx, U2 LM3671-3.3, U3 BQ24296, U4 USBLC6-4SC6

Commit message: sch wip
Parts:
- removed C17: 100u, symbol Device:CP
- added C17: 20u, Capacitors_SMD:C_1206, symbol Device:C
- added J3: V_3.3, Connector_PinHeader_2.54mm:PinHeader_1x02_P2.54mm_Vertical, symbol Connector_Generic:Conn_01x02
- added J4: CHRG_OUT, Connector_PinHeader_2.54mm:PinHeader_1x02_P2.54mm_Vertical, symbol Connector_Generic:Conn_01x02
- added J5: V_USB, Connector_PinHeader_2.54mm:PinHeader_1x02_P2.54mm_Vertical, symbol Connector_Generic:Conn_01x02
- C1, C10, C11, C13, C15, C24, C4, C6, C8, C9: footprint (none) -> Capacitors_SMD:C_0402_NoSilk
- C12, C14, C16, C18, C19, C2, C20, C22, C25, C26, C3, C5, C7: footprint (none) -> Capacitors_SMD:C_0805
- C21: footprint (none) -> Capacitors_SMD:C_1206
- C23: value 100u -> 20u; footprint (none) -> Capacitors_SMD:C_1206
- J1: footprint (none) -> Connectors:USB_Micro-B
- J2: footprint (none) -> Connector_PinHeader_2.54mm:PinHeader_1x02_P2.54mm_Vertical
- L1: footprint (none) -> Inductors_SMD:L_1210_HandSoldering
- R1, R2, R3, R4, R5, R6: footprint (none) -> Resistors_SMD:R_0603
- TS1: footprint (none) -> Connector_PinHeader_1.27mm:PinHeader_1x02_P1.27mm_Vertical
- U1: footprint Package_QFP:LQFP-100_14x14mm_P0.5mm -> Housings_QFP:LQFP-100_14x14mm_Pitch0.5mm
- U2: footprint Package_TO_SOT_SMD:TSOT-23-5 -> TO_SOT_Packages_SMD:TSOT-23-5
- U3: footprint (none) -> Housings_DFN_QFN:QFN-24_4x4mm_Pitch0.5mm
- U4: footprint Package_TO_SOT_SMD:SOT-23-6 -> TO_SOT_Packages_SMD:SOT-23-6
Connections:
- wire segments 250 -> 251
Other:
- moved on the sheet: C16

Commit message: sch core done
Parts:
- added C28, C29: 10u, Capacitors_SMD:C_0805, symbol Device:C
- added C30, C31: 10nF, Capacitors_SMD:C_0805, symbol Device:C
- added C32, C33: 30pF, Capacitors_SMD:C_0805, symbol Device:C
- added R10, R11: 510, Resistors_SMD:R_0603, symbol Device:R
- added R8, R9: 22k, Resistors_SMD:R_0603, symbol Device:R
- added U5, U6: KXO-V97, Crystals:Crystal_SMD_7050-4pin_7.0x5.0mm, symbol core:KXO-V97
- BT1: footprint (none) -> Connector_PinSocket_2.54mm:PinSocket_1x02_P2.54mm_Vertical
- J2: footprint Connector_PinHeader_2.54mm:PinHeader_1x02_P2.54mm_Vertical -> Connector_PinHeader_1.27mm:PinHeader_1x02_P1.27mm_Vertical
- L2: footprint (none) -> Inductors:Inductor_Taiyo-Yuden_NR-40xx_HandSoldering
Connections:
- net BAT_OTG is gone; now on net +3V3: U3.8 (OTG)
- net BAT_PSEL is gone; now on net +3V3: U3.2 (PSEL)
- net +3V3: now also C30.1, C31.1, U5.4 (VCC), U6.4 (VCC)
- net GND: now also C28.2, C29.2, C30.2, C31.2, C32.2, C33.2, R8.2, R9.2, U5.2 (GND), U6.2 (GND)
- net USB_ID: now also U4.4 (IO3); no longer U4.6 (IO4)
- net at C21.1, J4.1 (Pin_1), L2.2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: now also C28.1, C29.1
- net at U1.12 (PH0): now also R10.1, R11.1
- net USB_D+: now reaches U4.3 (IO2)
- net USB_D+: now also J1.3 (D+)
- net USB_DM renamed USB_D-
- net USB_D-: now also U4.1 (IO1); no longer U4.4 (IO3)
- removed net USB_DP: J1.3 (D+), U4.1 (IO1)
- new net: C32.1, R10.2, U5.3 (OUT)
- new net: C33.1, R11.2, U6.3 (OUT)
- new net CRYST_1: R9.1, U6.1 (EN)
- new net CRYST_2: R8.1, U5.1 (EN)
- no-connect marks 5 -> 3
Other:
- moved on the sheet: C21, J4

Commit message: sch upd
Parts:
- U1: symbol core:STM32F427VITx -> core-rescue:STM32F427VITx-core
- U2: symbol core:LM3671-3.3 -> core-rescue:LM3671-3.3-core
- U3: symbol core:BQ24296 -> core-rescue:BQ24296-core
- U4: symbol core:USBLC6-4SC6 -> core-rescue:USBLC6-4SC6-core
- U5, U6: symbol core:KXO-V97 -> core-rescue:KXO-V97-core
Connections:
- no-connect marks 3 -> 4
Changed lines of the file:
@@
 $EndDescr
 $Comp
-L core:BQ24296 U3
+L core-rescue:BQ24296-core U3
 U 1 1 5C3BFCB9
 P 4350 750
+AR Path="/5C3BFCB9" Ref="U3"  Part="1"
+AR Path="/5C3BFBF8/5C3BFCB9" Ref="U3"  Part="1"
 F 0 "U3" H 3750 815 50  0000 C CNN
 F 1 "BQ24296" H 3750 724 50  0000 C CNN
@@
 	7100 550  600  550
 $Comp
-L core:LM3671-3.3 U2
+L core-rescue:LM3671-3.3-core U2
 U 1 1 5C3F0F04
 P 1550 3950
@@
 Battery charger & controller
 $Comp
-L core:STM32F427VITx U1
+L core-rescue:STM32F427VITx-core U1
 U 4 1 5C42716C
 P 9050 1750
@@
 	3200 4150 3300 4150
 $Comp
-L core:USBLC6-4SC6 U4
+L core-rescue:USBLC6-4SC6-core U4
 U 1 1 5C681E02
 P 5000 4750
@@
 	5600 4000 6000 4000
 $Comp
-L core:KXO-V97 U5
+L core-rescue:KXO-V97-core U5
 U 1 1 5C525BA3
 P 7950 4150
@@
 	7400 4150 7500 4150
 $Comp
-L core:KXO-V97 U6
+L core-rescue:KXO-V97-core U6
 U 1 1 5C68096E
 P 7950 5650
@@
 	6250 3800 6000 3800
 Connection ~ 6000 3800
+NoConn ~ 4500 4650
 $EndSCHEMATC

Commit message: new charger schematic
Parts:
- removed C19: 4.7u, Capacitors_SMD:C_0805, symbol Device:C
- removed C20: 47n, Capacitors_SMD:C_0805, symbol Device:C
- removed C21, C23: 20u, Capacitors_SMD:C_1206, symbol Device:C
- removed L2: 1uH, Inductors:Inductor_Taiyo-Yuden_NR-40xx_HandSoldering, symbol Device:L
- removed R1: 22k, Resistors_SMD:R_0603, symbol Device:R
- removed R5: R, Resistors_SMD:R_0603, symbol Device:R
- removed R6: RT2, Resistors_SMD:R_0603, symbol Device:R
- removed TS1: 103 NTC Thermistor R25=10k, Connector_PinHeader_1.27mm:PinHeader_1x02_P1.27mm_Vertical, symbol Connector_Generic:Conn_01x02
- removed U3: BQ24296, Housings_DFN_QFN:QFN-24_4x4mm_Pitch0.5mm, symbol core-rescue:BQ24296-core
- added D1: 2A, Diode_SMD:D_2010_5025Metric, symbol Device:D_Schottky
- added F1: MF-SM100, Fuse:Fuse_Bourns_MF-SM_9.5x6.71mm, symbol Device:Fuse
- added U3: MCP73831-2-OT, Package_TO_SOT_SMD:SOT-23-5, symbol Battery_Management:MCP73831-2-OT
- added U7: DW01-P, Package_TO_SOT_SMD:SOT-23-6, symbol core-rescue:DW01-P
- added U8: 8205, Package_SO:TSSOP-8_4.4x3mm_P0.65mm, symbol core-rescue:8205
- C12: value 1u -> 10u
- C14: value 8.2u -> 10u
- C17: value 20u -> 100n; footprint Capacitors_SMD:C_1206 -> Capacitor_SMD:C_0402_1005Metric
- R2: value 22k -> 2k; footprint Resistors_SMD:R_0603 -> Resistor_SMD:R_0603_1608Metric_Pad1.05x0.95mm_HandSolder
- R3: value 22k -> 100; footprint Resistors_SMD:R_0603 -> Resistor_SMD:R_0603_1608Metric_Pad1.05x0.95mm_HandSolder
- R4: value RT1 -> 1k; footprint Resistors_SMD:R_0603 -> Resistor_SMD:R_0603_1608Metric_Pad1.05x0.95mm_HandSolder
Connections:
- net BAT_INT is gone; now on net +BATT: R3.1
- net +3V3: no longer R2.2, R3.2
- net +BATT: now also C28.1, C29.1, J4.1 (Pin_1), D1.1 (K), F1.1, U3.3 (VBAT); no longer BT1.1 (+)
- net BAT_CE: now also U3.1 (STAT)
- net GND: now also R2.2, R4.1, U3.2 (VSS), U8.6 (S2), U8.7 (S2); no longer BT1.2 (-), C17.2
- net VBUS: now also C14.1, U3.4 (VDD); no longer C17.1
- net at R4.2: now also U7.2 (CS)
- net BAT_SCL: no longer names the net of R2.1
- net BAT_SCL: now also U3.5 (PROG)
- new net: BT1.1 (+), F1.2
- new net: BT1.2 (-), C17.2, D1.2 (A), U7.6 (GND), U8.2 (S1), U8.3 (S1)
- new net: U7.1 (OD), U8.4 (G1)
- new net: U7.3 (OC), U8.5 (G2)
- new net: C17.1, R3.2, U7.5 (VCC)
- no-connect marks 4 -> 5
Other:
- note removed: "B57164-K 103-J"
- note removed: "RT1 and RT2\npage 26 in bq24296 datasheet"
- moved on the sheet: BT1, C22, C28, C29, J4

Commit message: pcb upd
Parts:
- C12, C14, C16, C18, C2, C22, C25, C26, C28, C29, C3, C30, C31, C32, C33, C5, C7: footprint Capacitors_SMD:C_0805 -> Capacitor_SMD:C_0805_2012Metric
- C17: footprint Capacitor_SMD:C_0402_1005Metric -> Capacitor_SMD:C_0805_2012Metric
- F1: value MF-SM100 -> MF-MSMF110; footprint Fuse:Fuse_Bourns_MF-SM_9.5x6.71mm -> Fuse:Fuse_1812_4532Metric_Pad1.30x3.40mm_HandSolder
- U4: footprint TO_SOT_Packages_SMD:SOT-23-6 -> Package_TO_SOT_SMD:SOT-23-6
Changed lines of the file:
@@
 F 0 "C22" H 3115 1246 50  0000 L CNN
 F 1 "10u" H 3115 1155 50  0000 L CNN
-F 2 "Capacitors_SMD:C_0805" H 3038 1050 50  0001 C CNN
+F 2 "Capacitor_SMD:C_0805_2012Metric" H 3038 1050 50  0001 C CNN
 F 3 "~" H 3000 1200 50  0001 C CNN
 	1    3000 1200
@@
 F 0 "C3" H 1065 4096 50  0000 L CNN
 F 1 "4.7u" H 1065 4005 50  0000 L CNN
-F 2 "Capacitors_SMD:C_0805" H 988 3900 50  0001 C CNN
+F 2 "Capacitor_SMD:C_0805_2012Metric" H 988 3900 50  0001 C CNN
 F 3 "~" H 950 4050 50  0001 C CNN
 	1    950  4050
@@
 F 0 "C16" H 2465 4096 50  0000 L CNN
 F 1 "10u" H 2465 4005 50  0000 L CNN
-F 2 "Capacitors_SMD:C_0805" H 2388 3900 50  0001 C CNN
+F 2 "Capacitor_SMD:C_0805_2012Metric" H 2388 3900 50  0001 C CNN
 F 3 "~" H 2350 4050 50  0001 C CNN
 	1    2350 4050
@@
 F 0 "C25" H 10285 1254 50  0000 R CNN
 F 1 "2.2u" H 10285 1345 50  0000 R CNN
-F 2 "Capacitors_SMD:C_0805" H 10438 1150 50  0001 C CNN
+F 2 "Capacitor_SMD:C_0805_2012Metric" H 10438 1150 50  0001 C CNN
 F 3 "~" H 10400 1300 50  0001 C CNN
 	1    10400 1300
@@
 F 0 "C26" H 10585 1254 50  0000 R CNN
 F 1 "2.2u" H 10585 1345 50  0000 R CNN
-F 2 "Capacitors_SMD:C_0805" H 10738 1150 50  0001 C CNN
+F 2 "Capacitor_SMD:C_0805_2012Metric" H 10738 1150 50  0001 C CNN
 F 3 "~" H 10700 1300 50  0001 C CNN
 	1    10700 1300
@@
 F 0 "C2" H 865 5946 50  0000 L CNN
 F 1 "1u" H 865 5855 50  0000 L CNN
-F 2 "Capacitors_SMD:C_0805" H 788 5750 50  0001 C CNN
+F 2 "Capacitor_SMD:C_0805_2012Metric" H 788 5750 50  0001 C CNN
 F 3 "~" H 750 5900 50  0001 C CNN
 	1    750  5900
@@
 F 0 "C5" H 1065 5946 50  0000 L CNN
 F 1 "1u" H 1065 5855 50  0000 L CNN
-F 2 "Capacitors_SMD:C_0805" H 988 5750 50  0001 C CNN
+F 2 "Capacitor_SMD:C_0805_2012Metric" H 988 5750 50  0001 C CNN
 F 3 "~" H 950 5900 50  0001 C CNN
 	1    950  5900
@@
 F 0 "C7" H 1265 5946 50  0000 L CNN
 F 1 "4.7u" H 1265 5855 50  0000 L CNN
-F 2 "Capacitors_SMD:C_0805" H 1188 5750 50  0001 C CNN
+F 2 "Capacitor_SMD:C_0805_2012Metric" H 1188 5750 50  0001 C CNN
 F 3 "~" H 1150 5900 50  0001 C CNN
 	1    1150 5900
@@
 F 0 "C18" H 3415 4046 50  0000 L CNN
 F 1 "1u" H 3415 3955 50  0000 L CNN
-F 2 "Capacitors_SMD:C_0805" H 3338 3850 50  0001 C CNN
+F 2 "Capacitor_SMD:C_0805_2012Metric" H 3338 3850 50  0001 C CNN
 F 3 "~" H 3300 4000 50  0001 C CNN
 	1    3300 4000
@@
 F 0 "U4" H 5250 4400 50  0000 C CNN
 F 1 "USBLC6-4SC6" H 5300 5100 50  0000 C CNN
-F 2 "TO_SOT_Packages_SMD:SOT-23-6" H 4250 5150 50  0001 C CNN
+F 2 "Package_TO_SOT_SMD:SOT-23-6" H 4250 5150 50  0001 C CNN
 F 3 "http://www2.st.com/resource/en/datasheet/CD00050750.pdf" H 5200 5100 50  0001 C CNN
 	1    5000 4750
@@
 F 0 "C28" H 3465 1246 50  0000 L CNN
 F 1 "10u" H 3465 1155 50  0000 L CNN
-F 2 "Capacitors_SMD:C_0805" H 3388 1050 50  0001 C CNN
+F 2 "Capacitor_SMD:C_0805_2012Metric" H 3388 1050 50  0001 C CNN
 F 3 "~" H 3350 1200 50  0001 C CNN
 	1    3350 1200
@@
 F 0 "C29" H 3665 1246 50  0000 L CNN
 F 1 "10u" H 3665 1155 50  0000 L CNN
-F 2 "Capacitors_SMD:C_0805" H 3588 1050 50  0001 C CNN
+F 2 "Capacitor_SMD:C_0805_2012Metric" H 3588 1050 50  0001 C CNN
 F 3 "~" H 3550 1200 50  0001 C CNN
 	1    3550 1200
@@
 F 0 "C32" H 8565 4396 50  0000 L CNN
 F 1 "30pF" H 8565 4305 50  0000 L CNN
-F 2 "Capacitors_SMD:C_0805" H 8488 4200 50  0001 C CNN
+F 2 "Capacitor_SMD:C_0805_2012Metric" H 8488 4200 50  0001 C CNN
 F 3 "~" H 8450 4350 50  0001 C CNN
 	1    8450 4350
@@
 F 0 "C30" H 7565 3746 50  0000 L CNN
 F 1 "10nF" H 7565 3655 50  0000 L CNN
-F 2 "Capacitors_SMD:C_0805" H 7488 3550 50  0001 C CNN
+F 2 "Capacitor_SMD:C_0805_2012Metric" H 7488 3550 50  0001 C CNN
 F 3 "~" H 7450 3700 50  0001 C CNN
 	1    7450 3700
@@
 F 0 "C33" H 8565 5896 50  0000 L CNN
 F 1 "30pF" H 8565 5805 50  0000 L CNN
-F 2 "Capacitors_SMD:C_0805" H 8488 5700 50  0001 C CNN
+F 2 "Capacitor_SMD:C_0805_2012Metric" H 8488 5700 50  0001 C CNN
 F 3 "~" H 8450 5850 50  0001 C CNN
 	1    8450 5850
@@
 F 0 "C31" H 7565 5246 50  0000 L CNN
 F 1 "10nF" H 7565 5155 50  0000 L CNN
-F 2 "Capacitors_SMD:C_0805" H 7488 5050 50  0001 C CNN
+F 2 "Capacitor_SMD:C_0805_2012Metric" H 7488 5050 50  0001 C CNN
 F 3 "~" H 7450 5200 50  0001 C CNN
 	1    7450 5200
@@
 F 0 "C17" H 4865 2446 50  0000 L CNN
 F 1 "100n" H 4865 2355 50  0000 L CNN
-F 2 "Capacitor_SMD:C_0402_1005Metric" H 4788 2250 50  0001 C CNN
+F 2 "Capacitor_SMD:C_0805_2012Metric" H 4788 2250 50  0001 C CNN
 F 3 "~" H 4750 2400 50  0001 C CNN
 	1    4750 2400
@@
 P 4200 1750
 F 0 "F1" V 4003 1750 50  0000 C CNN
-F 1 "MF-SM100" V 4094 1750 50  0000 C CNN
-F 2 "Fuse:Fuse_Bourns_MF-SM_9.5x6.71mm" V 4130 1750 50  0001 C CNN
+F 1 "MF-MSMF110" V 4094 1750 50  0000 C CNN
+F 2 "Fuse:Fuse_1812_4532Metric_Pad1.30x3.40mm_HandSolder" V 4130 1750 50  0001 C CNN
 F 3 "~" H 4200 1750 50  0001 C CNN
 	1    4200 1750
@@
 F 0 "C14" H 3215 4046 50  0000 L CNN
 F 1 "10u" H 3215 3955 50  0000 L CNN
-F 2 "Capacitors_SMD:C_0805" H 3138 3850 50  0001 C CNN
+F 2 "Capacitor_SMD:C_0805_2012Metric" H 3138 3850 50  0001 C CNN
 F 3 "~" H 3100 4000 50  0001 C CNN
 	1    3100 4000
@@
 F 0 "C12" H 1015 1346 50  0000 L CNN
 F 1 "10u" H 1015 1255 50  0000 L CNN
-F 2 "Capacitors_SMD:C_0805" H 938 1150 50  0001 C CNN
+F 2 "Capacitor_SMD:C_0805_2012Metric" H 938 1150 50  0001 C CNN
 F 3 "~" H 900 1300 50  0001 C CNN
 	1    900  1300
