File: sch/core/power.sch (KiCad schematic (older format))
At the start: 52 parts, among them J1 USB_B_Micro, J2 Reset, J3 V_3.3, J4 CHRG_OUT, J5 V_USB, U1 STM32F427VITx, U2 LM3671-3.3, U3 MCP73831-2-OT, U4 USBLC6-4SC6, U5 KXO-V97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

Commit message: PCB v.2 completed
Parts:
- U1: symbol core-rescue:STM32F427VITx-core -> core-rescue:STM32F427VITx-core-core-rescue
- U2: symbol core-rescue:LM3671-3.3-core -> core-rescue:LM3671-3.3-core-core-rescue
- U4: symbol core-rescue:USBLC6-4SC6-core -> core-rescue:USBLC6-4SC6-core-core-rescue
- U5, U6: symbol core-rescue:KXO-V97-core -> core-rescue:KXO-V97-core-core-rescue
- U7: symbol core-rescue:DW01-P -> core-rescue:DW01-P-core-rescue
- U8: symbol core-rescue:8205 -> core-rescue:8205-core-rescue
Connections:
- net +3V3: now also C31.1, U6.4 (VCC)
Changed lines of the file:
@@
 	7100 550  600  550
 $Comp
-L core-rescue:LM3671-3.3-core U2
+L core-rescue:LM3671-3.3-core-core-rescue U2
 U 1 1 5C3F0F04
 P 1550 3950
@@
 Battery charger & controller
 $Comp
-L core-rescue:STM32F427VITx-core U1
+L core-rescue:STM32F427VITx-core-core-rescue U1
 U 4 1 5C42716C
 P 9050 1750
@@
 	3200 4150 3300 4150
 $Comp
-L core-rescue:USBLC6-4SC6-core U4
+L core-rescue:USBLC6-4SC6-core-core-rescue U4
 U 1 1 5C681E02
 P 5000 4750
@@
 	5600 4000 6000 4000
 $Comp
-L core-rescue:KXO-V97-core U5
+L core-rescue:KXO-V97-core-core-rescue U5
 U 1 1 5C525BA3
 P 7950 4150
@@
 	7400 4150 7500 4150
 $Comp
-L core-rescue:KXO-V97-core U6
+L core-rescue:KXO-V97-core-core-rescue U6
 U 1 1 5C68096E
 P 7950 5650
@@
 L power:+3.3V #PWR0137
 U 1 1 5C680991
-P 8100 5150
-F 0 "#PWR0137" H 8100 5000 50  0001 C CNN
-F 1 "+3.3V" H 8115 5323 50  0000 C CNN
-F 2 "" H 8100 5150 50  0001 C CNN
-F 3 "" H 8100 5150 50  0001 C CNN
-	1    8100 5150
+P 8050 5150
+F 0 "#PWR0137" H 8050 5000 50  0001 C CNN
+F 1 "+3.3V" H 8065 5323 50  0000 C CNN
+F 2 "" H 8050 5150 50  0001 C CNN
+F 3 "" H 8050 5150 50  0001 C CNN
+	1    8050 5150
 	1    0    0    -1
 $EndComp
@@
 	3000 1000 3000 1050
 $Comp
-L core-rescue:DW01-P U7
+L core-rescue:DW01-P-core-rescue U7
 U 1 1 5CBF741E
 P 5350 2400
@@
 $EndComp
 $Comp
-L core-rescue:8205 U8
+L core-rescue:8205-core-rescue U8
 U 1 1 5CBF8908
 P 6200 2500
+AR Path="/5CBF8908" Ref="U8"  Part="1"
+AR Path="/5C3BFBF8/5CBF8908" Ref="U8"  Part="1"
 F 0 "U8" H 6350 2250 50  0000 C CNN
 F 1 "8205" H 6300 2750 50  0000 C CNN
@@
 	900  1800 1200 1800
 Connection ~ 1200 1800
+Wire Wire Line
+	7950 5250 7950 5200
+Wire Wire Line
+	8050 5150 8050 5200
+Wire Wire Line
+	8050 5200 7950 5200
+Connection ~ 7950 5200
+Wire Wire Line
+	7950 5200 7950 5000
 $EndSCHEMATC
