File: sch/core/display.sch (KiCad schematic (older format))
At the start: 2 parts, among them J6 Conn_01x09

Commit message: sch core done
Parts:
- removed J6: Conn_01x09, Connector_PinHeader_2.54mm:PinHeader_1x09_P2.54mm_Vertical, symbol Connector_Generic:Conn_01x09
- added J6: Conn_01x18, core:ILI9341_18Pin, symbol Connector_Generic:Conn_01x18
- added Q1: BSS138, TO_SOT_Packages_SMD:SOT-23, symbol Transistor_FET:BSS138
- added R7: R_BACKLIGHT, Resistors_SMD:R_0805, symbol Device:R
Connections:
- wire segments 10 -> 26
- no-connect marks 0 -> 4
Other:
- moved on the sheet: C27
Changed lines of the file:
@@
 Comment4 ""
 $EndDescr
-Text HLabel 5500 3850 0    50   Input ~ 0
+Text HLabel 6500 3550 0    50   Input ~ 0
 MISO
-Text HLabel 5500 3750 0    50   Input ~ 0
-LED
-Text HLabel 5500 3650 0    50   Input ~ 0
+Text HLabel 6500 3150 0    50   Input ~ 0
 SCK
-Text HLabel 5500 3550 0    50   Input ~ 0
+Text HLabel 6500 3450 0    50   Input ~ 0
 MOSI
-Text HLabel 5500 3450 0    50   Input ~ 0
+Text HLabel 6500 3250 0    50   Input ~ 0
 DC
-Text HLabel 5500 3350 0    50   Input ~ 0
+Text HLabel 6500 3050 0    50   Input ~ 0
 RST
-Text HLabel 5500 3250 0    50   Input ~ 0
+Text HLabel 6500 3350 0    50   Input ~ 0
 CS
-$Comp
-L Connector_Generic:Conn_01x09 J6
-U 1 1 5C4DC60F
-P 5700 3450
-F 0 "J6" H 5780 3492 50  0000 L CNN
-F 1 "Conn_01x09" H 5780 3401 50  0000 L CNN
-F 2 "Connector_PinHeader_2.54mm:PinHeader_1x09_P2.54mm_Vertical" H 5700 3450 50  0001 C CNN
-F 3 "~" H 5700 3450 50  0001 C CNN
-	1    5700 3450
-	1    0    0    -1
-$EndComp
 $Comp
 L Device:C C27
 U 1 1 5C4DC6F4
-P 5000 3100
-F 0 "C27" H 5115 3146 50  0000 L CNN
-F 1 "20u" H 5115 3055 50  0000 L CNN
-F 2 "Capacitors_SMD:C_0805" H 5038 2950 50  0001 C CNN
-F 3 "~" H 5000 3100 50  0001 C CNN
-	1    5000 3100
-	1    0    0    -1
+P 5750 3700
+F 0 "C27" H 5865 3746 50  0000 L CNN
+F 1 "20u" H 5865 3655 50  0000 L CNN
+F 2 "Capacitors_SMD:C_0805" H 5788 3550 50  0001 C CNN
+F 3 "~" H 5750 3700 50  0001 C CNN
+	1    5750 3700
+	1    0    0    1
 $EndComp
 $Comp
 L power:+3.3V #PWR0129
 U 1 1 5C4DC7FF
-P 5000 2850
-F 0 "#PWR0129" H 5000 2700 50  0001 C CNN
-F 1 "+3.3V" H 5015 3023 50  0000 C CNN
-F 2 "" H 5000 2850 50  0001 C CNN
-F 3 "" H 5000 2850 50  0001 C CNN
-	1    5000 2850
+P 5750 3950
+F 0 "#PWR0129" H 5750 3800 50  0001 C CNN
+F 1 "+3.3V" H 5765 4123 50  0000 C CNN
+F 2 "" H 5750 3950 50  0001 C CNN
+F 3 "" H 5750 3950 50  0001 C CNN
+	1    5750 3950
+	1    0    0    1
+$EndComp
+Wire Wire Line
+	5750 3950 5750 3900
+$Comp
+L power:GND #PWR0130
+U 1 1 5C4DC874
+P 5750 3450
+F 0 "#PWR0130" H 5750 3200 50  0001 C CNN
+F 1 "GND" H 5755 3277 50  0000 C CNN
+F 2 "" H 5750 3450 50  0001 C CNN
+F 3 "" H 5750 3450 50  0001 C CNN
+	1    5750 3450
+	1    0    0    1
+$EndComp
+Wire Wire Line
+	5750 3450 5750 3500
+Connection ~ 5750 3900
+Wire Wire Line
+	5750 3900 5750 3850
+Wire Wire Line
+	6050 3500 6050 3650
+Connection ~ 5750 3500
+Wire Wire Line
+	5750 3500 5750 3550
+Wire Wire Line
+	6050 3750 6050 3850
+Wire Wire Line
+	5750 3500 6050 3500
+Wire Wire Line
+	5750 3900 6050 3900
+$Comp
+L Connector_Generic:Conn_01x18 J6
+U 1 1 5C4FC248
+P 6700 3750
+F 0 "J6" H 6780 3742 50  0000 L CNN
+F 1 "Conn_01x18" H 6780 3651 50  0000 L CNN
+F 2 "core:ILI9341_18Pin" H 6700 3750 50  0001 C CNN
+F 3 "~" H 6700 3750 50  0001 C CNN
+	1    6700 3750
+	1    0    0    -1
+$EndComp
+$Comp
+L power:GND #PWR0131
+U 1 1 5C4FC327
+P 5750 3000
+F 0 "#PWR0131" H 5750 2750 50  0001 C CNN
+F 1 "GND" H 5755 2827 50  0000 C CNN
+F 2 "" H 5750 3000 50  0001 C CNN
+F 3 "" H 5750 3000 50  0001 C CNN
+	1    5750 3000
 	1    0    0    -1
 $EndComp
 Wire Wire Line
-	5000 2850 5000 2900
+	5750 3000 5750 2950
+Wire Wire Line
+	5750 2950 6500 2950
+Wire Wire Line
+	6050 3650 6500 3650
+Wire Wire Line
+	6050 3750 6500 3750
+NoConn ~ 6500 4650
+NoConn ~ 6500 4550
+NoConn ~ 6500 4450
+NoConn ~ 6500 4350
+Wire Wire Line
+	6500 3850 6050 3850
+Connection ~ 6050 3850
+Wire Wire Line
+	6050 3850 6050 3900
+Wire Wire Line
+	6500 3950 6450 3950
+Wire Wire Line
+	6450 3950 6450 4050
+Wire Wire Line
+	6450 4250 6500 4250
+Wire Wire Line
+	6500 4150 6450 4150
+Connection ~ 6450 4150
+Wire Wire Line
+	6450 4150 6450 4250
+Wire Wire Line
+	6500 4050 6450 4050
+Connection ~ 6450 4050
+Wire Wire Line
+	6450 4050 6450 4100
 $Comp
-L power:GND #PWR0130
-U 1 1 5C4DC874
-P 5000 3350
-F 0 "#PWR0130" H 5000 3100 50  0001 C CNN
-F 1 "GND" H 5005 3177 50  0000 C CNN
-F 2 "" H 5000 3350 50  0001 C CNN
-F 3 "" H 5000 3350 50  0001 C CNN
-	1    5000 3350
+L Transistor_FET:BSS138 Q1
+U 1 1 5C4FCE3D
+P 5800 4750
+F 0 "Q1" H 6005 4796 50  0000 L CNN
+F 1 "BSS138" H 6005 4705 50  0000 L CNN
+F 2 "TO_SOT_Packages_SMD:SOT-23" H 6000 4675 50  0001 L CIN
+F 3 "https://www.fairchildsemi.com/datasheets/BS/BSS138.pdf" H 5800 4750 50  0001 L CNN
+	1    5800 4750
+	1    0    0    -1
+$EndComp
+Connection ~ 6450 4100
+Wire Wire Line
+	6450 4100 6450 4150
+$Comp
+L power:GND #PWR0132
+U 1 1 5C4FD085
+P 5900 5050
+F 0 "#PWR0132" H 5900 4800 50  0001 C CNN
+F 1 "GND" H 5905 4877 50  0000 C CNN
+F 2 "" H 5900 5050 50  0001 C CNN
+F 3 "" H 5900 5050 50  0001 C CNN
+	1    5900 5050
+	-1   0    0    -1
+$EndComp
+Wire Wire Line
+	5900 5050 5900 4950
+$Comp
+L Device:R R7
+U 1 1 5C4FD507
+P 5900 4350
+F 0 "R7" H 5970 4396 50  0000 L CNN
+F 1 "R_BACKLIGHT" H 5970 4305 50  0000 L CNN
+F 2 "Resistors_SMD:R_0805" V 5830 4350 50  0001 C CNN
+F 3 "~" H 5900 4350 50  0001 C CNN
+	1    5900 4350
 	1    0    0    -1
 $EndComp
 Wire Wire Line
-	5000 3350 5000 3300
-Connection ~ 5000 2900
+	5900 4550 5900 4500
 Wire Wire Line
-	5000 2900 5000 2950
+	5900 4200 5900 4100
 Wire Wire Line
-	5300 3300 5300 3150
-Wire Wire Line
-	5300 3150 5500 3150
-Connection ~ 5000 3300
-Wire Wire Line
-	5000 3300 5000 3250
-Wire Wire Line
-	5300 3050 5300 2900
-Wire Wire Line
-	5300 3050 5500 3050
-Wire Wire Line
-	5000 3300 5300 3300
-Wire Wire Line
-	5000 2900 5300 2900
+	5900 4100 6450 4100
+Text HLabel 5600 4750 0    50   Input ~ 0
+LED
 $EndSCHEMATC

Commit message: pcb upd
Parts:
- C27: footprint Capacitors_SMD:C_0805 -> Capacitor_SMD:C_0805_2012Metric
Changed lines of the file:
@@
 F 0 "C27" H 5865 3746 50  0000 L CNN
 F 1 "20u" H 5865 3655 50  0000 L CNN
-F 2 "Capacitors_SMD:C_0805" H 5788 3550 50  0001 C CNN
+F 2 "Capacitor_SMD:C_0805_2012Metric" H 5788 3550 50  0001 C CNN
 F 3 "~" H 5750 3700 50  0001 C CNN
 	1    5750 3700
